Commit message: realsense camera d435i 부착 완료(urdf, mesh, 런치파일 수정.)

File: srdf/ur_robotiq.srdf.xacro (robot description, xacro)
@@ -114,3 +114,47 @@
   <disable_collisions link1="$(arg prefix)ur_to_robotiq_link" link2="$(arg prefix)wrist_2_link" reason="Never" />
   <disable_collisions link1="$(arg prefix)ur_to_robotiq_link" link2="$(arg prefix)wrist_3_link" reason="Adjacent" />
+  <!-- ==================== 카메라 브라켓 충돌 비활성화 ==================== -->
+  <!-- 카메라 브라켓과 tool0, wrist 링크들 -->
+  <disable_collisions link1="$(arg prefix)camera_bracket_link" link2="$(arg prefix)tool0" reason="Adjacent" />
+  <disable_collisions link1="$(arg prefix)camera_bracket_link" link2="$(arg prefix)wrist_1_link" reason="Never" />
+  <disable_collisions link1="$(arg prefix)camera_bracket_link" link2="$(arg prefix)wrist_2_link" reason="Never" />
+  <disable_collisions link1="$(arg prefix)camera_bracket_link" link2="$(arg prefix)wrist_3_link" reason="Never" />
+  <!-- 카메라 브라켓과 그리퍼 어댑터 (브라켓에서 그리퍼가 연결됨) -->
+  <disable_collisions link1="$(arg prefix)camera_bracket_link" link2="$(arg prefix)ur_to_robotiq_link" reason="Adjacent" />
+  <!-- 카메라 브라켓과 그리퍼 링크들 -->
+  <disable_collisions link1="$(arg prefix)camera_bracket_link" link2="$(arg prefix)robotiq_85_base_link" reason="Never" />
+  <disable_collisions link1="$(arg prefix)camera_bracket_link" link2="$(arg prefix)robotiq_85_left_knuckle_link" reason="Never" />
+  <disable_collisions link1="$(arg prefix)camera_bracket_link" link2="$(arg prefix)robotiq_85_right_knuckle_link" reason="Never" />
+  <disable_collisions link1="$(arg prefix)camera_bracket_link" link2="$(arg prefix)robotiq_85_left_finger_link" reason="Never" />
+  <disable_collisions link1="$(arg prefix)camera_bracket_link" link2="$(arg prefix)robotiq_85_right_finger_link" reason="Never" />
+  <!-- 그리퍼 마운팅 포인트와 어댑터 -->
+  <disable_collisions link1="$(arg prefix)gripper_mounting_point" link2="$(arg prefix)camera_bracket_link" reason="Adjacent" />
+  <disable_collisions link1="$(arg prefix)gripper_mounting_point" link2="$(arg prefix)ur_to_robotiq_link" reason="Adjacent" />
+  <disable_collisions link1="$(arg prefix)gripper_mounting_point" link2="$(arg prefix)tool0" reason="Never" />
+  <!-- ==================== RealSense D435i 카메라 충돌 비활성화 ==================== -->
+  <!-- 카메라 마운팅 포인트 -->
+  <disable_collisions link1="$(arg prefix)camera_mounting_point" link2="$(arg prefix)camera_bracket_link" reason="Adjacent" />
+  <disable_collisions link1="$(arg prefix)camera_mounting_point" link2="$(arg prefix)camera_link" reason="Adjacent" />
+  <!-- 카메라 링크와 주변 링크들 -->
+  <disable_collisions link1="$(arg prefix)camera_link" link2="$(arg prefix)camera_bracket_link" reason="Never" />
+  <disable_collisions link1="$(arg prefix)camera_link" link2="$(arg prefix)camera_mounting_point" reason="Adjacent" />
+  <disable_collisions link1="$(arg prefix)camera_link" link2="$(arg prefix)tool0" reason="Never" />
+  <disable_collisions link1="$(arg prefix)camera_link" link2="$(arg prefix)wrist_1_link" reason="Never" />
+  <disable_collisions link1="$(arg prefix)camera_link" link2="$(arg prefix)wrist_2_link" reason="Never" />
+  <disable_collisions link1="$(arg prefix)camera_link" link2="$(arg prefix)wrist_3_link" reason="Never" />
+  <disable_collisions link1="$(arg prefix)camera_link" link2="$(arg prefix)ur_to_robotiq_link" reason="Never" />
+  <disable_collisions link1="$(arg prefix)camera_link" link2="$(arg prefix)robotiq_85_base_link" reason="Never" />
+  <!-- 카메라 optical frame들은 물리적 충돌 체크 불필요 -->
+  <disable_collisions link1="$(arg prefix)camera_depth_frame" link2="$(arg prefix)camera_link" reason="Adjacent" />
+  <disable_collisions link1="$(arg prefix)camera_depth_optical_frame" link2="$(arg prefix)camera_depth_frame" reason="Adjacent" />
+  <disable_collisions link1="$(arg prefix)camera_color_frame" link2="$(arg prefix)camera_depth_frame" reason="Adjacent" />
+  <disable_collisions link1="$(arg prefix)camera_color_optical_frame" link2="$(arg prefix)camera_color_frame" reason="Adjacent" />
+  <disable_collisions link1="$(arg prefix)camera_infra1_frame" link2="$(arg prefix)camera_depth_frame" reason="Adjacent" />
+  <disable_collisions link1="$(arg prefix)camera_infra1_optical_frame" link2="$(arg prefix)camera_infra1_frame" reason="Adjacent" />
+  <disable_collisions link1="$(arg prefix)camera_infra2_frame" link2="$(arg prefix)camera_depth_frame" reason="Adjacent" />
+  <disable_collisions link1="$(arg prefix)camera_infra2_optical_frame" link2="$(arg prefix)camera_infra2_frame" reason="Adjacent" />
+  <disable_collisions link1="$(arg prefix)camera_accel_frame" link2="$(arg prefix)camera_link" reason="Adjacent" />
+  <disable_collisions link1="$(arg prefix)camera_accel_optical_frame" link2="$(arg prefix)camera_accel_frame" reason="Adjacent" />
+  <disable_collisions link1="$(arg prefix)camera_gyro_frame" link2="$(arg prefix)camera_link" reason="Adjacent" />
+  <disable_collisions link1="$(arg prefix)camera_gyro_optical_frame" link2="$(arg prefix)camera_gyro_frame" reason="Adjacent" />
 </robot>

File: urdf/ur5e_robotiq_2f85.urdf.xacro (robot description, xacro)
@@ -10,4 +10,8 @@
   <!-- import main UR macro & Robotiq macros -->
   <xacro:include filename="$(find ur_description)/urdf/ur_macro.xacro"/>
+  <!-- 카메라 브라켓 어댑터 -->
+  <xacro:include filename="$(find ur_picking)/urdf/camera_bracket_adapter.urdf.xacro" />
+  <!-- RealSense D435i 공식 매크로 -->
+  <xacro:include filename="$(find realsense2_description)/urdf/_d435i.urdf.xacro" />
   <!-- Use local adapter to avoid duplicate gripper base link -->
   <xacro:include filename="$(find ur_picking)/urdf/ur_to_robotiq_adapter.urdf.xacro" />
@@ -127,8 +131,19 @@
     <origin xyz="0 0 0" rpy="0 0 0" />
   </xacro:ur_robot>
-  <!-- Robotiq 2F-85 어댑터 + 그리퍼 부착 (UR tool0 기준) -->
+  <!-- ===================== 카메라 브라켓 부착 (tool0에 직접) ===================== -->
+  <xacro:camera_bracket_adapter
+    prefix="$(arg tf_prefix)"
+    parent="$(arg tf_prefix)tool0" />
+  <!-- ===================== RealSense D435i 카메라 부착 (브라켓에) ===================== -->
+  <xacro:sensor_d435i
+    parent="$(arg tf_prefix)camera_mounting_point"
+    name="$(arg tf_prefix)camera"
+    use_nominal_extrinsics="true">
+    <origin xyz="0 0 0" rpy="0 0 0"/>
+  </xacro:sensor_d435i>
+  <!-- ===================== Robotiq 2F-85 어댑터 + 그리퍼 부착 (브라켓에) ===================== -->
   <xacro:ur_to_robotiq
     prefix="$(arg tf_prefix)"
-    parent="$(arg tf_prefix)tool0"
+    parent="$(arg tf_prefix)gripper_mounting_point"
     child="$(arg tf_prefix)robotiq_85_base_link" />
   <xacro:robotiq_gripper
@@ -147,5 +162,5 @@
     </gazebo>
     <gazebo>
-      <plugin filename="libign_ros2_control-system.so" name="ign_ros2_control::IgnitionROS2ControlPlugin">
+      <plugin filename="libgz_ros2_control-system.so" name="gz_ros2_control::GazeboSimROS2ControlPlugin">
         <parameters>$(arg simulation_controllers)</parameters>
         <controller_manager_node_name>$(arg tf_prefix)controller_manager</controller_manager_node_name>

File: urdf/ur_to_robotiq_adapter.urdf.xacro (robot description, xacro)
@@ -1,11 +1,4 @@
 <?xml version="1.0" encoding="utf-8"?>
 <robot xmlns:xacro="http://ros.org/wiki/xacro">
-  <!--
-    Local copy of ur_to_robotiq adapter macro, simplified to avoid
-    creating the gripper base link twice.
-    Original macro signature is kept for compatibility, but the 'child'
-    link and associated joint are not created here. The Robotiq macro
-    itself will create robotiq_85_base_link.
-  -->
   <xacro:macro name="ur_to_robotiq" params="prefix parent child rotation:=^|${0.0}">
     <!-- Adapter joint from UR tool0 (parent) to intermediate adapter link -->
@@ -35,9 +28,4 @@
       </inertial>
     </link>
-    <!-- NOTE:
-      We intentionally do NOT create a second joint/link to 'child' here.
-      The Robotiq macro will create 'robotiq_85_base_link' itself. Creating
-      it here as well leads to duplicate link names and URDF parse errors.
-    -->
   </xacro:macro>
 </robot>
